Commit message: add heading_frame, some launch files, support for zedm

File: zed-ros-wrapper/zed_wrapper/urdf/zedm.urdf (robot description, URDF)
Before this commit: robot zedm_camera, 7 links, 6 joints
Links:
- removed link base_link
- added link zed_base_link
Joints:
- joint zed_camera_center_joint: parent base_link -> zed_base_link
